Commit message: Updated to 3 imus kinda working ish.

File: hbo/urdf/suit.urdf.xacro (robot description, xacro)
@@ -4,5 +4,5 @@
     name="hbosuit">
     <xacro:include filename="$(find hbo)/urdf/common.urdf.xacro" />
-    <xacro:include filename="$(find hbo)/urdf/sensors/um7.urdf.xacro" />
+    <xacro:include filename="$(find hbo)/urdf/body/upper_body_imu.urdf.xacro" />
     <!-- Note: Base Link is the back of the skull, right where the Zelmet strap is. -->
     <!-- Physical Constant Macros -->
@@ -10,66 +10,74 @@
     <xacro:property name="M_41deg" value="0.7155849933176751265387132150803312" />
     <xacro:property name="M_16deg" value="0.279252680319092732307790522958" />
-    <!-- IMU placement relative to base_link -->
-    <xacro:property name="imu_x" value=".0381" />
+	<!-- IMU placement relative to chest -->
+    <xacro:property name="imu_x" value="0" />
     <xacro:property name="imu_y" value="0" />
-    <xacro:property name="imu_z" value=".1016" />
+    <xacro:property name="imu_z" value="0" />
     <xacro:property name="imu_roll" value="0" />
-    <xacro:property name="imu_pitch" value="-${M_41deg}" />
+    <xacro:property name="imu_pitch" value="0" />
     <xacro:property name="imu_yaw" value="0" />
-     <!-- ZED placement relative to base_link -->
-    <xacro:property name="zed_x" value="0.2286" />
-    <xacro:property name="zed_y" value="0.0" />
-    <xacro:property name="zed_z" value="0.0508" />
-    <xacro:property name="zed_roll" value="0" />
-    <xacro:property name="zed_pitch" value="${M_16deg}" />
-    <xacro:property name="zed_yaw" value="0" />
-    <!-- Main body of Helmet -->
-    <link name="base_link">
-        <inertial>
-            <mass value="0.162" />
-            <origin xyz="0 0 0" />
-            <inertia  ixx="0.2" ixy="0.0"  ixz="0.0"  iyy="0.2"  iyz="0.0"  izz="0.2" />
-        </inertial>
-        <visual>
-            <origin xyz="0.1016 0 0.0508" rpy="0 0 0" />
-            <geometry>
-                 <cylinder radius="0.1016" length="0.1016" />
-             </geometry>
-            <material name="Blue"/>
-        </visual>
-        <collision>
-            <origin xyz="0.1016 0 0.0508" rpy="0 0 0" />
-            <geometry>
-                 <cylinder radius="0.1016" length="0.1016" />
-             </geometry>
-        </collision>
+ 	<!-- Body dimensions -->
+    <xacro:property name="w_shoulder" value=".3048" />
+    <xacro:property name="l_upper_arm" value=".3048" />
+    <xacro:property name="l_forearm" value=".2667" />
+	<xacro:property name="r_upper_arm" value=".0424" />
+    <xacro:property name="r_forearm" value="0.03436155221" />
+	<xacro:property name="l_chest" value="0.1016" />
+<!-- Chest -->
+    <link name="origin_link">
     </link>
-    <!-- Visor -->
-    <joint name="visor_joint" type="fixed" >
-        <parent link="base_link" />
-        <child link="visor_link" />
-    </joint>
-	<link name="visor_link">
-        <visual>
-            <origin xyz="0.1778 0 0.0127" rpy="0 0 0" />
-            <geometry>
-                 <box size=".1016 .1651 .0254" />
-             </geometry>
-            <material name="Blue"/>
-        </visual>
-        <collision>
-            <origin xyz="0.1778 0 0.0127" rpy="0 0 0" />
-            <geometry>
-                 <box size=".1016 .1651 .0254" />
-             </geometry>
-        </collision>
-    </link>
-    <!-- IMU -->
+	<!-- IMU -->
     <xacro:um7_imu_v0
-        name="imu"
-        parent="base_link">
+        name="imu_chest"
+		parent ="origin_link"
+		child ="chest_link">
         <origin
             xyz="${imu_x} ${imu_y} ${imu_z}"
             rpy="${imu_roll} ${imu_pitch} ${imu_yaw}" />
     </xacro:um7_imu_v0>
+    <!-- Chest -->
+    <link name="chest_link">
+        <visual>
+            <origin xyz="0 0 ${w_shoulder/4}" rpy="0 0 0" />
+            <geometry>
+                 <box size="${w_shoulder} ${w_shoulder/2} ${w_shoulder/2}" length="${l_chest}" />
+             </geometry>
+            <material name="DarkGrey"/>
+        </visual>
+    </link>
+    <!-- IMU -->
+    <xacro:um7_imu_v0
+        name="imu_upper_right_arm"
+		parent ="chest_link"
+		child ="right_upper_arm_link">
+            <origin xyz="${w_shoulder/2} 0 .1" rpy="0 0 0" />
+    </xacro:um7_imu_v0>
+	<!-- Upper arm -->
+	<link name="right_upper_arm_link">
+        <visual>
+            <origin xyz="${l_upper_arm/2} 0 0" rpy="0 ${M_PI/2} 0" />
+            <geometry>
+                 <cylinder radius="${r_upper_arm}" length="${l_upper_arm}" />
+             </geometry>
+            <material name="DarkGrey"/>
+        </visual>
+   </link>
+    <!-- IMU -->
+    <xacro:um7_imu_v0
+        name="imu_right_forearm"
+		parent ="right_upper_arm_link"
+		child = "right_forearm_link">
+        <origin
+            xyz="${l_upper_arm} 0 0" rpy="0 0 0" />
+    </xacro:um7_imu_v0> 0
+	<!-- Forearm -->
+	<link name="right_forearm_link">
+        <visual>
+           <origin xyz="${l_forearm/2} 0 0" rpy="0 ${M_PI/2} 0" />
+            <geometry>
+                 <cylinder radius="${r_forearm}" length="${l_forearm}" />
+             </geometry>
+            <material name="DarkGrey"/>
+        </visual>
+    </link>
 </robot>

Commit message: redid links, figured out how to publish JointStates, 5 days til Boeing Demo!

File: hbo/urdf/suit.urdf.xacro (robot description, xacro)
@@ -9,6 +9,6 @@
     <xacro:property name="M_PI"    value="3.1415926535897931" />
     <xacro:property name="M_41deg" value="0.7155849933176751265387132150803312" />
-    <xacro:property name="M_16deg" value="0.279252680319092732307790522958" />
-	<!-- IMU placement relative to chest -->
+    <xacro:property name="M_16deg" value="0.2792526803190927a32307790522958" />
+    <!-- IMU placement relative to chest -->
     <xacro:property name="imu_x" value="0" />
     <xacro:property name="imu_y" value="0" />
@@ -17,29 +17,41 @@
     <xacro:property name="imu_pitch" value="0" />
     <xacro:property name="imu_yaw" value="0" />
- 	<!-- Body dimensions -->
+    <!-- Body dimensions -->
     <xacro:property name="w_shoulder" value=".3048" />
     <xacro:property name="l_upper_arm" value=".3048" />
     <xacro:property name="l_forearm" value=".2667" />
-	<xacro:property name="r_upper_arm" value=".0424" />
+    <xacro:property name="r_upper_arm" value=".0424" />
     <xacro:property name="r_forearm" value="0.03436155221" />
-	<xacro:property name="l_chest" value="0.1016" />
-<!-- Chest -->
+    <xacro:property name="l_chest" value="0.1016" />
+    <!-- Chest -->
     <link name="origin_link">
     </link>
-	<!-- IMU -->
-    <xacro:um7_imu_v0
-        name="imu_chest"
-		parent ="origin_link"
-		child ="chest_link">
-        <origin
-            xyz="${imu_x} ${imu_y} ${imu_z}"
-            rpy="${imu_roll} ${imu_pitch} ${imu_yaw}" />
-    </xacro:um7_imu_v0>
-    <!-- Chest -->
+     <joint name="chest_yaw" type="continuous">
+         <parent link="origin_link"/>
+         <child link="chest_yaw_link"/>
+         <axis xyz="0 0 1"/>
+         <origin xyz="0 0 0"/>
+    </joint>
+    <link name="chest_yaw_link">
+    </link>
+    <joint name="chest_pitch" type="continuous">
+         <parent link="chest_yaw_link"/>
+         <child link="chest_pitch_link"/>
+         <axis xyz="0 1 0"/>
+         <origin xyz="0 0 0"/>
+    </joint>
+    <link name="chest_pitch_link">
+    </link>
+    <joint name="chest_roll" type="continuous">
+         <parent link="chest_pitch_link"/>
+         <child link="chest_link"/>
+         <axis xyz="1 0 0"/>
+         <origin xyz="0 0 0"/>
+    </joint>
     <link name="chest_link">
         <visual>
-            <origin xyz="0 0 ${w_shoulder/4}" rpy="0 0 0" />
+            <origin xyz="0 0 0" rpy="0 0 0" />
             <geometry>
-                 <box size="${w_shoulder} ${w_shoulder/2} ${w_shoulder/2}" length="${l_chest}" />
+                 <box size="${w_shoulder/2} ${w_shoulder} ${w_shoulder/2}" length="${l_chest}" />
              </geometry>
             <material name="DarkGrey"/>
@@ -48,13 +60,37 @@
     <!-- IMU -->
     <xacro:um7_imu_v0
-        name="imu_upper_right_arm"
-		parent ="chest_link"
-		child ="right_upper_arm_link">
-            <origin xyz="${w_shoulder/2} 0 .1" rpy="0 0 0" />
+        name="imu_chest"
+        parent="chest_link">
+        <origin
+            xyz="${imu_x} ${imu_y} ${imu_z}"
+            rpy="${imu_roll} ${imu_pitch} ${imu_yaw}" />
     </xacro:um7_imu_v0>
-	<!-- Upper arm -->
-	<link name="right_upper_arm_link">
+    <!-- Shoulder -->
+     <joint name="right_shoulder_yaw" type="continuous">
+         <parent link="chest_link"/>
+         <child link="rshoulder_yaw_link"/>
+         <axis xyz="0 0 1"/>
+         <origin xyz="0 ${-w_shoulder/2} 0" rpy="0 0 ${-M_PI/2}"/>
+       </joint>
+    <link name="rshoulder_yaw_link">
+    </link>
+    <joint name="right_shoulder_pitch" type="continuous">
+         <parent link="rshoulder_yaw_link"/>
+         <child link="rshoulder_pitch_link"/>
+         <axis xyz="0 1 0"/>
+         <origin xyz="0 0 0"/>
+       </joint>
+    <link name="rshoulder_pitch_link">
+    </link>
+    <joint name="right_shoulder_roll" type="continuous">
+         <parent link="rshoulder_pitch_link"/>
+         <child link="right_upper_arm_link"/>
+         <axis xyz="1 0 0"/>
+         <origin xyz="0 0 0"/>
+       </joint>
+    <!-- Upper arm -->
+    <link name="right_upper_arm_link">
         <visual>
-            <origin xyz="${l_upper_arm/2} 0 0" rpy="0 ${M_PI/2} 0" />
+            <origin xyz="${w_shoulder/2} 0 0" rpy="0 ${M_PI/2} 0" />
             <geometry>
                  <cylinder radius="${r_upper_arm}" length="${l_upper_arm}" />
@@ -65,12 +101,19 @@
     <!-- IMU -->
     <xacro:um7_imu_v0
-        name="imu_right_forearm"
-		parent ="right_upper_arm_link"
-		child = "right_forearm_link">
+        name="imu_upper_right_arm"
+        parent="right_upper_arm_link">
         <origin
-            xyz="${l_upper_arm} 0 0" rpy="0 0 0" />
-    </xacro:um7_imu_v0> 0
-	<!-- Forearm -->
-	<link name="right_forearm_link">
+            xyz="${imu_x} ${imu_y} ${imu_z}"
+            rpy="${imu_roll} ${imu_pitch} ${imu_yaw}" />
+    </xacro:um7_imu_v0>
+    <!-- Elbow -->
+    <joint name="right_elbow" type="continuous">
+         <parent link="right_upper_arm_link"/>
+         <child link="right_forearm_link"/>
+         <axis xyz="0 1 0"/>
+         <origin xyz="${l_upper_arm} 0 0"/>
+    </joint>
+    <!-- Forearm -->
+    <link name="right_forearm_link">
         <visual>
            <origin xyz="${l_forearm/2} 0 0" rpy="0 ${M_PI/2} 0" />
@@ -81,3 +124,11 @@
         </visual>
     </link>
+    <!-- IMU -->
+    <xacro:um7_imu_v0
+        name="imu_right_forearm"
+        parent="right_forearm_link">
+        <origin
+            xyz="${imu_x} ${imu_y} ${imu_z}"
+            rpy="${imu_roll} ${imu_pitch} ${imu_yaw}" />
+    </xacro:um7_imu_v0>
 </robot>

Commit message: Added extra arm for demo

File: hbo/urdf/suit.urdf.xacro (robot description, xacro)
@@ -132,3 +132,69 @@
             rpy="${imu_roll} ${imu_pitch} ${imu_yaw}" />
     </xacro:um7_imu_v0>
+<!-- Shoulder -->
+     <joint name="left_shoulder_yaw" type="continuous">
+         <parent link="chest_link"/>
+         <child link="lshoulder_yaw_link"/>
+         <axis xyz="0 0 1"/>
+         <origin xyz="0 ${w_shoulder/2} 0" rpy="0 0 ${-M_PI/2}"/>
+       </joint>
+    <link name="lshoulder_yaw_link">
+    </link>
+    <joint name="left_shoulder_pitch" type="continuous">
+         <parent link="lshoulder_yaw_link"/>
+         <child link="lshoulder_pitch_link"/>
+         <axis xyz="0 1 0"/>
+         <origin xyz="0 0 0"/>
+       </joint>
+    <link name="lshoulder_pitch_link">
+    </link>
+    <joint name="left_shoulder_roll" type="continuous">
+         <parent link="lshoulder_pitch_link"/>
+         <child link="left_upper_arm_link"/>
+         <axis xyz="1 0 0"/>
+         <origin xyz="0 0 0"/>
+       </joint>
+    <!-- Upper arm -->
+    <link name="left_upper_arm_link">
+        <visual>
+            <origin xyz="${-w_shoulder/2} 0 0" rpy="0 ${M_PI/2} 0" />
+            <geometry>
+                 <cylinder radius="${r_upper_arm}" length="${l_upper_arm}" />
+             </geometry>
+            <material name="DarkGrey"/>
+        </visual>
+   </link>
+    <!-- IMU -->
+    <xacro:um7_imu_v0
+        name="imu_upper_left_arm"
+        parent="origin_link">
+        <origin
+            xyz="${imu_x} ${imu_y} ${imu_z}"
+            rpy="${imu_roll} ${imu_pitch} ${imu_yaw}" />
+    </xacro:um7_imu_v0>
+    <!-- Elbow -->
+    <joint name="left_elbow" type="continuous">
+         <parent link="left_upper_arm_link"/>
+         <child link="left_forearm_link"/>
+         <axis xyz="0 1 0"/>
+         <origin xyz="${-l_upper_arm} 0 0"/>
+    </joint>
+    <!-- Forearm -->
+    <link name="left_forearm_link">
+        <visual>
+           <origin xyz="${-l_forearm/2} 0 0" rpy="0 ${M_PI/2} 0" />
+            <geometry>
+                 <cylinder radius="${r_forearm}" length="${l_forearm}" />
+             </geometry>
+            <material name="DarkGrey"/>
+        </visual>
+    </link>
+    <!-- IMU -->
+    <xacro:um7_imu_v0
+        name="imu_left_forearm"
+        parent="origin_link">
+        <origin
+            xyz="${imu_x} ${imu_y} ${imu_z}"
+            rpy="${imu_roll} ${imu_pitch} ${imu_yaw}" />
+    </xacro:um7_imu_v0>
 </robot>

Commit message: Got 4 IMUs working with the zelmet model

File: hbo/urdf/suit.urdf.xacro (robot description, xacro)
@@ -5,4 +5,5 @@
     <xacro:include filename="$(find hbo)/urdf/common.urdf.xacro" />
     <xacro:include filename="$(find hbo)/urdf/body/upper_body_imu.urdf.xacro" />
+    <xacro:include filename="$(find zelmet)/urdf/zelmet.urdf.xacro" />
     <!-- Note: Base Link is the back of the skull, right where the Zelmet strap is. -->
     <!-- Physical Constant Macros -->
@@ -61,9 +62,32 @@
     <xacro:um7_imu_v0
         name="imu_chest"
-        parent="origin_link">
+        parent="chest_link">
         <origin
             xyz="${imu_x} ${imu_y} ${imu_z}"
             rpy="${imu_roll} ${imu_pitch} ${imu_yaw}" />
     </xacro:um7_imu_v0>
+    <joint name="helmet_yaw" type="continuous">
+         <parent link="chest_link"/>
+         <child link="helmet_yaw_link"/>
+         <axis xyz="0 0 1"/>
+         <origin xyz="0 0 .2"/>
+    </joint>
+    <link name="helmet_yaw_link">
+    </link>
+    <joint name="helmet_pitch" type="continuous">
+         <parent link="helmet_yaw_link"/>
+         <child link="helmet_pitch_link"/>
+         <axis xyz="0 1 0"/>
+         <origin xyz="0 0 0"/>
+    </joint>
+    <link name="helmet_pitch_link">
+    </link>
+    <joint name="helmet_roll" type="continuous">
+         <parent link="helmet_pitch_link"/>
+         <child link="helmet_link"/>
+         <axis xyz="1 0 0"/>
+         <origin xyz="0 0 0"/>
+    </joint>
+    <xacro:zelmet />
     <!-- Shoulder -->
      <joint name="right_shoulder_yaw" type="continuous">
@@ -102,5 +126,5 @@
     <xacro:um7_imu_v0
         name="imu_upper_right_arm"
-        parent="origin_link">
+        parent="right_upper_arm_link">
         <origin
             xyz="${imu_x} ${imu_y} ${imu_z}"
@@ -127,5 +151,5 @@
     <xacro:um7_imu_v0
         name="imu_right_forearm"
-        parent="origin_link">
+        parent="right_forearm_link">
         <origin
             xyz="${imu_x} ${imu_y} ${imu_z}"

File: zelmet/urdf/zelmet.urdf.xacro (robot description, xacro)
@@ -2,7 +2,7 @@
 <robot
     xmlns:xacro="http://www.ros.org/wiki/xacro"
-    name="gigatron">
+    name="zelmet">
     <xacro:include filename="$(find zelmet)/urdf/sensors/zed.urdf.xacro" />
-    <xacro:include filename="$(find zelmet)/urdf/common.urdf.xacro" />
+    <!-- <xacro:include filename="$(find zelmet)/urdf/common.urdf.xacro" /> -->
     <xacro:include filename="$(find zelmet)/urdf/sensors/um7.urdf.xacro" />
     <!-- Note: Base Link is the back of the skull, right where the Zelmet strap is. -->
@@ -16,5 +16,6 @@
     <xacro:property name="imu_z" value=".1016" />
     <xacro:property name="imu_roll" value="0" />
-    <xacro:property name="imu_pitch" value="-${M_41deg}" />
+    <!-- <xacro:property name="imu_pitch" value="-${M_41deg}" /> -->
+    <xacro:property name="imu_pitch" value="0" />
     <xacro:property name="imu_yaw" value="0" />
      <!-- ZED placement relative to base_link -->
@@ -22,9 +23,10 @@
     <xacro:property name="zed_y" value="0.0" />
     <xacro:property name="zed_z" value="0.0508" />
-    <xacro:property name="zed_roll" value="0" />
-    <xacro:property name="zed_pitch" value="${M_16deg}" />
+    <xacro:property name="zed_roll" value="0" /> <!--
+    <xacro:property name="zed_pitch" value="${M_16deg}" /> -->
+    <xacro:property name="zed_pitch" value="0" />
     <xacro:property name="zed_yaw" value="0" />
     <!-- Main body of Helmet -->
-    <link name="base_link">
+    <link name="helmet_link">
         <inertial>
             <mass value="0.162" />
@@ -48,5 +50,5 @@
     <!-- Visor -->
     <joint name="visor_joint" type="fixed" >
-        <parent link="base_link" />
+        <parent link="helmet_link" />
         <child link="visor_link" />
     </joint>
@@ -68,6 +70,6 @@
     <!-- IMU -->
     <xacro:um7_imu_v0
-        name="imu"
-        parent="base_link">
+        name="imu_zelmet"
+        parent="helmet_link">
         <origin
             xyz="${imu_x} ${imu_y} ${imu_z}"
@@ -77,5 +79,5 @@
     <xacro:zed_v0
         name="zed"
-        parent="base_link">
+        parent="helmet_link">
         <origin
             xyz="${zed_x} ${zed_y} ${zed_z}"
